Commit message: added coriolos, smoothed out contact, derivative check passed for 1e-6 noise

File: data/robosimian_caesar_new_pinocchio.urdf (robot description, URDF)
Before this commit: robot robosimian_caesar, 33 links, 32 joints
Links:
- added link virtual0, mass 0
- added link virtual1, mass 0
- added link virtual2, mass 0
- link limb1_link7: geometry collision cylinder length=0.146 radius=0.05; visual mesh filename=stl_0_3/top_limb.stl scale=0.001 0.001 0.001
- link limb2_link7: geometry collision cylinder length=0.146 radius=0.05; visual mesh filename=stl_0_3/bottom_limb.stl scale=0.001 0.001 0.001
- link limb3_link7: geometry collision cylinder length=0.146 radius=0.05; visual mesh filename=stl_0_3/bottom_limb.stl scale=0.001 0.001 0.001
- link limb4_link7: geometry collision cylinder length=0.146 radius=0.05; visual mesh filename=stl_0_3/top_limb.stl scale=0.001 0.001 0.001
Joints:
- added joint torso_a: type revolute, parent virtual2, child torso, origin xyz=0.0 0.0 0.0 rpy=0.00000 -0.00000 0.00000, axis 0 1 0, limit lower=-3 upper=3 effort=1000.0 velocity=100
- added joint torso_x: type prismatic, parent virtual0, child virtual1, origin xyz=0.0 0.0 0.0 rpy=0.00000 -0.00000 0.00000, axis 1 0 0, limit lower=-1000 upper=1000 effort=100000.0 velocity=0
- added joint torso_z: type prismatic, parent virtual1, child virtual2, origin xyz=0.0 0.0 0.0 rpy=0.00000 -0.00000 0.00000, axis 0 0 1, limit lower=-1000 upper=1000 effort=100000.0 velocity=0
- joint limb1_joint0: type revolute -> fixed
- joint limb1_joint1: type revolute -> fixed
- joint limb1_joint3: type revolute -> fixed
- joint limb1_joint5: type revolute -> fixed
- joint limb1_joint7: limit lower=-3.1415 upper=3.1415 effort=1000.0 velocity=0.5 -> lower=0 upper=0 effort=0.0 velocity=0
- joint limb2_joint0: type revolute -> fixed
- joint limb2_joint1: type revolute -> fixed
- joint limb2_joint3: type revolute -> fixed
- joint limb2_joint5: type revolute -> fixed
- joint limb2_joint7: limit lower=-3.1415 upper=3.1415 effort=1000.0 velocity=0.5 -> lower=0 upper=0 effort=0.0 velocity=0
- joint limb3_joint0: type revolute -> fixed
- joint limb3_joint1: type revolute -> fixed
- joint limb3_joint3: type revolute -> fixed
- joint limb3_joint5: type revolute -> fixed
- joint limb3_joint7: limit lower=-3.1415 upper=3.1415 effort=1000.0 velocity=0.5 -> lower=0 upper=0 effort=0.0 velocity=0
- joint limb4_joint0: type revolute -> fixed
- joint limb4_joint1: type revolute -> fixed
- joint limb4_joint3: type revolute -> fixed
- joint limb4_joint5: type revolute -> fixed
- joint limb4_joint7: limit lower=-3.1415 upper=3.1415 effort=1000.0 velocity=0.5 -> lower=0 upper=0 effort=0.0 velocity=0
