Commit message: recent changes

File: data/robosimian_caesar_new_all_active.urdf (robot description, URDF)
Before this commit: robot robosimian_caesar, 33 links, 32 joints
Links:
- link limb1_link7: geometry collision cylinder length=0.15 radius=0.05; visual mesh filename=stl_0_3/ankle_mm.STL scale=0.001 0.001 0.001
- link limb2_link7: geometry collision cylinder length=0.15 radius=0.05; visual mesh filename=stl_0_3/ankle_mm.STL scale=0.001 0.001 0.001
- link limb3_link7: geometry collision cylinder length=0.15 radius=0.05; visual mesh filename=stl_0_3/ankle_mm.STL scale=0.001 0.001 0.001
- link limb4_link7: geometry collision cylinder length=0.15 radius=0.05; visual mesh filename=stl_0_3/ankle_mm.STL scale=0.001 0.001 0.001
